File: pppadpcbv1 acrheron type c.kicad_pcb (KiCad board)
At the start: 2 copper layers, 59 parts, among them SW1 MXSwitch, SW10 MXSwitch, SW11 MXSwitch, SW12 MXSwitch, SW13 MXSwitch, SW14 MXSwitch, SW15 MXSwitch, SW16 MXSwitch, SW17 MXSwitch, SW18 MXSwitch, SW19 MXSwitch, SW2 MXSwitch, SW20 MXSwitch, SW3 MXSwitch, SW4 MXSwitch, SW5 MXSwitch, SW6 MXSwitch, SW7 MXSwitch, SW8 MXSwitch, SW9 MXSwitch, U1 ATmega32U4-AU, Y1 16MHz

Commit message: 7/4/2020
Fixed usbc
Parts:
- removed REF**: TYPE-C-31-M-12, acheron_Connectors:TYPE-C-31-M-12
- added J1: TYPE-C-31-M12_13, acheron_Connectors:TYPE-C-31-M-12, F.Cu at (-214.3, -142.9)
- C1: value 100n -> 100nF
- moved C3 217.5 mm to (75.8, 67.8)
- moved C7 217.5 mm to (50.2, 41.0)
- moved C8 217.5 mm to (85.7, 75.6)
- moved D1 217.5 mm to (65.0, 54.6)
- moved D10 217.5 mm to (90.9, 79.1)
- moved D15 217.5 mm to (70.8, 54.6)
- moved D16 217.5 mm to (55.5, 41.2)
- moved D18 217.5 mm to (65.0, 47.9)
- moved D2 217.5 mm to (75.3, 64.7)
- moved D20 217.5 mm to (70.8, 47.9)
- moved D3 217.5 mm to (59.3, 47.9)
- moved D4 217.5 mm to (70.8, 58.0)
- moved D7 217.5 mm to (61.2, 41.2)
- moved SWP1 217.5 mm to (68.9, 42.9)
- moved U1 217.5 mm to (85.4, 66.9)
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Connections:
- C1 pad 1: Net-(C1-Pad1) -> GND
- R5 pad 1: Net-(C1-Pad1) -> Net-(R5-Pad1)
- SWP1 pad 1: Net-(C1-Pad1) -> Net-(R5-Pad1)
Other:
- board outline added: 81 x 100 mm
