File: pppadpcbv1 acrheron type c.sch (KiCad schematic (older format))
At the start: 59 parts, among them J1 TYPE-C-31-M12_13, SW1 MXSwitch, SW10 MXSwitch, SW11 MXSwitch, SW12 MXSwitch, SW13 MXSwitch, SW14 MXSwitch, SW15 MXSwitch, SW16 MXSwitch, SW17 MXSwitch, SW18 MXSwitch, SW19 MXSwitch, SW2 MXSwitch, SW20 MXSwitch, SW3 MXSwitch, SW4 MXSwitch, SW5 MXSwitch, SW6 MXSwitch, SW7 MXSwitch, SW8 MXSwitch, SW9 MXSwitch, U1 ATmega32U4-AU, Y1 16MHz

Commit message: 7/4/2020
Fixed usbc
Parts:
- C1: value 100n -> 100nF
- J1: footprint acheronConnectors:TYPE-C-31-M-12 -> acheron_Connectors:TYPE-C-31-M-12
Connections:
- net GND: now also C1.1
- net at R5.1, SWP1.1: no longer C1.1
Other:
- moved on the sheet: R5
Changed lines of the file:
@@
 U 1 1 5EFB331D
 P 2200 3750
-F 0 "C1" V 2050 3850 50  0000 C CNN
-F 1 "100n" V 2150 3900 50  0000 C CNN
+F 0 "C1" V 2000 3750 50  0000 C CNN
+F 1 "100nF" V 2100 3750 50  0000 C CNN
 F 2 "Capacitor_SMD:C_0805_2012Metric_Pad1.15x1.40mm_HandSolder" H 2200 3750 50  0001 C CNN
 F 3 "~" H 2200 3750 50  0001 C CNN
@@
 L power:GND #PWR02
 U 1 1 5EFB9F0F
-P 2200 4150
-F 0 "#PWR02" H 2200 3900 50  0001 C CNN
-F 1 "GND" H 2200 4000 50  0000 C CNN
-F 2 "" H 2200 4150 50  0001 C CNN
-F 3 "" H 2200 4150 50  0001 C CNN
-	1    2200 4150
+P 2050 4150
+F 0 "#PWR02" H 2050 3900 50  0001 C CNN
+F 1 "GND" H 2050 4000 50  0000 C CNN
+F 2 "" H 2050 4150 50  0001 C CNN
+F 3 "" H 2050 4150 50  0001 C CNN
+	1    2050 4150
 	1    0    0    -1
 $EndComp
@@
 Wire Wire Line
 	2200 3850 2200 3950
-Wire Wire Line
-	2200 3950 2050 3950
-Connection ~ 2200 3950
 $Comp
 L Device:C_Small C5
@@
 L Device:R_Small R5
 U 1 1 5F0B0EAC
-P 2200 4050
-F 0 "R5" H 2050 4100 50  0000 L CNN
-F 1 "330" H 2000 4000 50  0000 L CNN
-F 2 "Resistor_SMD:R_1206_3216Metric_Pad1.42x1.75mm_HandSolder" H 2200 4050 50  0001 C CNN
-F 3 "~" H 2200 4050 50  0001 C CNN
-	1    2200 4050
+P 2050 4050
+F 0 "R5" H 1900 4100 50  0000 L CNN
+F 1 "330" H 1850 4000 50  0000 L CNN
+F 2 "Resistor_SMD:R_1206_3216Metric_Pad1.42x1.75mm_HandSolder" H 2050 4050 50  0001 C CNN
+F 3 "~" H 2050 4050 50  0001 C CNN
+	1    2050 4050
 	1    0    0    -1
 $EndComp
@@
 F 0 "J1" H 1607 7217 50  0000 C CNN
 F 1 "TYPE-C-31-M12_13" H 1607 7126 50  0000 C CNN
-F 2 "acheronConnectors:TYPE-C-31-M-12" V 1000 5850 50  0001 C CNN
+F 2 "acheron_Connectors:TYPE-C-31-M-12" V 1000 5850 50  0001 C CNN
 F 3 "https://www.usb.org/sites/default/files/documents/usb_type-c.zip" H 1700 5850 50  0001 C CNN
 	1    1500 5800
@@
 Text GLabel 2300 6150 2    50   Output ~ 0
 D+
+$Comp
+L power:GND #PWR?
+U 1 1 5F01852F
+P 2200 3950
+F 0 "#PWR?" H 2200 3700 50  0001 C CNN
+F 1 "GND" H 2200 3800 50  0000 C CNN
+F 2 "" H 2200 3950 50  0001 C CNN
+F 3 "" H 2200 3950 50  0001 C CNN
+	1    2200 3950
+	1    0    0    -1
+$EndComp
 $EndSCHEMATC
